Commit message: update_last_friday

File: pointgrey_camera_driver/pointgrey_camera_description/urdf/camera_tiago.urdf.xacro (robot description, xacro)
@@ -1,11 +1,12 @@
 <?xml version="1.0"?>
-<robot xmlns:xacro="http://www.ros.org/wiki/xacro" name="bumblebee2">
+<robot xmlns:xacro="http://www.ros.org/wiki/xacro" name="flea3">
   <link name="world"/>
-  <xacro:include filename="$(find pointgrey_camera_description)/urdf/pointgrey_bumblebee2.urdf.xacro" />
-  <BB2-08S2C-38 frame="bumblebee2" name="bumblebee2" />
+  <xacro:include filename="$(find pointgrey_camera_description)/urdf/pointgrey_flea3.urdf.xacro" />
+  <pointgrey_flea3 frame="flea3" name="flea3" camera_x="0.0754" camera_y="0.029" camera_z="0.035" camera_mass="0.085"
+                   hfov="1.0471975512" fps="60" width="640" height="512"/>
   <joint name="world_camera_joint" type="fixed">
     <origin xyz="0 0 0.470" rpy="0 0.4014 0" />
     <parent link="world" />
-    <child link="bumblebee2" />
+    <child link="flea3" />
   </joint>
 </robot>
